Commit message: Added Gazebo World

File: description/robot_core.xacro (robot description, xacro)
@@ -43,4 +43,7 @@
     </xacro:inertial_box>
   </link>
+  <gazebo reference="chassis">
+    <material>Gazebo/Blue</material>
+  </gazebo>
   <!-- LEFT WHEEL LINK -->
   <joint name="wheel_l_joint" type="continuous">
@@ -52,5 +55,5 @@
   <link name="wheel_l">
     <visual>
-      <origin xyz="0 0 0.1" />
+      <origin xyz="0 0 0.0" />
       <geometry>
         <cylinder radius="0.05" length="0.04" />
@@ -59,5 +62,5 @@
     </visual>
     <collision>
-      <origin xyz="0 0 0.1" />
+      <origin xyz="0 0 0.0" />
       <geometry>
         <cylinder radius="0.05" length="0.04" />
@@ -68,4 +71,7 @@
     </xacro:inertial_cylinder>
   </link>
+  <gazebo reference="wheel_l">
+    <material>Gazebo/Black</material>
+  </gazebo>
   <!-- RIGHT WHEEL LINK -->
   <joint name="wheel_r_joint" type="continuous">
@@ -77,5 +83,5 @@
   <link name="wheel_r">
     <visual>
-      <origin xyz="0 0 0.1" />
+      <origin xyz="0 0 0.0" />
       <geometry>
         <cylinder radius="0.05" length="0.04" />
@@ -84,5 +90,5 @@
     </visual>
     <collision>
-      <origin xyz="0 0 0.1" />
+      <origin xyz="0 0 0.0" />
       <geometry>
         <cylinder radius="0.05" length="0.04" />
@@ -93,4 +99,7 @@
     </xacro:inertial_cylinder>
   </link>
+  <gazebo reference="wheel_r">
+    <material>Gazebo/Black</material>
+  </gazebo>
   <!-- CASTER WHEEL LINK -->
   <joint name="wheel_c_joint" type="fixed">
@@ -115,3 +124,8 @@
     </xacro:inertial_sphere>
   </link>
+  <gazebo reference="wheel_c">
+    <material>Gazebo/Red</material>
+    <mu1 value="0.001"/>
+    <mu2 value="0.001"/>
+  </gazebo>
 </robot>
